File: WRadioLogo/WRadioLogo.kicad_pcb (KiCad board)
At the start: 2 copper layers, 100 x 100 mm, 99 parts, among them J1 TYPE-C-31-M-12, J2 Conn_01x04_Pin, J3 Conn_01x03_Pin, SW1 SW_Push, SW2 SW_Push, SW3 SW_Push, U1 STM32F030F4Px, U2 AMS1117-3.3

Commit message: nieuwe patronen + helderheid wip
Parts:
- removed R2: 10kΩ, Resistor_SMD:R_0805_2012Metric_Pad1.20x1.40mm_HandSolder
- removed SW2: SW_Push, Button_Switch_SMD:SW_SPST_FSMSM
Connections:
- U1 pad 1: BOOT -> GND
Routing:
- net BOOT: track 23.0 -> 0.00 mm
- net +3.3V: track 147.9 -> 146.0 mm
- net GND: track 924.4 -> 922.8 mm
Other:
- board text added: "WRadio - 23/05/25"
- board text removed: "WRadio - 19/04/25"
