File: WRadioLogo/WRadioLogo.kicad_sch (KiCad schematic)
At the start: 99 parts, among them J1 TYPE-C-31-M-12, J2 Conn_01x04_Pin, J3 Conn_01x03_Pin, SW1 SW_Push, SW2 SW_Push, SW3 SW_Push, U1 STM32F030F4Px, U2 AMS1117-3.3

Commit message: nieuwe patronen + helderheid wip
Parts:
- removed R2: 10kΩ, Resistor_SMD:R_0805_2012Metric_Pad1.20x1.40mm_HandSolder, symbol Device:R
- removed SW2: SW_Push, Button_Switch_SMD:SW_SPST_FSMSM, symbol Switch:SW_Push
Connections:
- net BOOT is gone; now on net GND: U1.1 (BOOT0)
Other:
- note removed: "Boot Button"
- moved on the sheet: C5, R1, SW1
